File: hardware/dual_spi_ports.kicad_sch (KiCad schematic)
At the start: 22 parts

Commit message: Add PDF schematics
Parts:
- C15: value (none) -> 0.1uF; footprint (none) -> Capacitor_SMD:C_0402_1005Metric
- C16, C17, C18, C19, C20, C21: value (none) -> 220pF; footprint (none) -> Capacitor_SMD:C_0402_1005Metric
- J2, J3: value (none) -> SM07B-GHS-TB; footprint (none) -> Connector_JST:JST_GH_SM07B-GHS-TB_1x07-1MP_P1.25mm_Horizontal
- R22, R27: value (none) -> 100k; footprint (none) -> Resistor_SMD:R_0402_1005Metric
- R23, R24, R25, R26, R30, R31, R32, R33: value (none) -> 100; footprint (none) -> Resistor_SMD:R_0402_1005Metric
- R28, R29: value (none) -> 10k; footprint (none) -> Resistor_SMD:R_0402_1005Metric
- U5: value (none) -> 74HC244; footprint (none) -> Package_SO:TSSOP-20_4.4x6.5mm_P0.65mm
Other:
- company: (none) -> LGR
- title: (none) -> ESP32 SPI hub - SPI ports
