File: hardware/esp32-spi-hub.kicad_sch (KiCad schematic)
At the start: 58 parts

Commit message: Add PDF schematics
Parts:
- C1, C10, C12, C3, C5, C7: value (none) -> 0.1uF; footprint (none) -> Capacitor_SMD:C_0402_1005Metric
- C11, C2, C4, C8: value (none) -> 10uF; footprint (none) -> Capacitor_Tantalum_SMD:CP_EIA-3216-18_Kemet-A
- C13, C14: value (none) -> 1nF; footprint (none) -> Capacitor_SMD:C_0402_1005Metric
- C6: value (none) -> 22uF; footprint (none) -> Capacitor_SMD:C_0603_1608Metric
- C9: value (none) -> 10uF; footprint (none) -> Capacitor_SMD:C_0402_1005Metric
- D1: value (none) -> SS34; footprint (none) -> Diode_SMD:D_SMA
- D2: value (none) -> YE; footprint (none) -> LED_SMD:LED_0603_1608Metric
- D3: value (none) -> GN; footprint (none) -> LED_SMD:LED_0603_1608Metric
- D4: value (none) -> BU; footprint (none) -> LED_SMD:LED_0603_1608Metric
- FB1: value (none) -> 100 @ 100MHz; footprint (none) -> Resistor_SMD:R_0805_2012Metric
- H1, H2, H3, H4, H5, H6: value (none) -> MountingHole; footprint (none) -> MountingHole:MountingHole_3mm
- J1: value (none) -> EXT_HEADER; footprint (none) -> Connector_PinHeader_2.00mm:PinHeader_1x08_P2.00mm_Vertical
- P1: value (none) -> USB_C_Plug_USB2.0; footprint (none) -> Connector_USB:USB_C_Receptacle_Palconn_UTC16-G
- Q1: value (none) -> AO3401A; footprint (none) -> Package_TO_SOT_SMD:SOT-23
- Q2, Q3: value (none) -> S8050; footprint (none) -> Package_TO_SOT_SMD:SOT-23
- R1: value (none) -> 4.7k; footprint (none) -> Resistor_SMD:R_0402_1005Metric
- R10, R11, R12, R13, R14, R2, R9: value (none) -> 100; footprint (none) -> Resistor_SMD:R_0402_1005Metric
- R15, R16: value (none) -> 5.1k; footprint (none) -> Resistor_SMD:R_0402_1005Metric
- R17, R21: value (none) -> 470; footprint (none) -> Resistor_SMD:R_0402_1005Metric
- R18, R19, R20: value (none) -> 1k; footprint (none) -> Resistor_SMD:R_0402_1005Metric
- R3, R4, R5, R6: value (none) -> 12k; footprint (none) -> Resistor_SMD:R_0402_1005Metric
- R7, R8: value (none) -> DNP; footprint (none) -> Resistor_SMD:R_0402_1005Metric
- RN1: value (none) -> 1k; footprint (none) -> Resistor_SMD:R_Array_Convex_4x0603
- SW1, SW2: value (none) -> SW_Push; footprint (none) -> Button_Switch_SMD:SW_SPST_B3U-1000P-B
- U1: value (none) -> AMS1117-3.3; footprint (none) -> Package_TO_SOT_SMD:SOT-223-3_TabPin2
- U2: value (none) -> CP2102-GMR; footprint (none) -> Package_DFN_QFN:QFN-28-1EP_5x5mm_P0.5mm_EP3.35x3.35mm
- U3: value (none) -> ESP32-WROOM-32UE-N16; footprint (none) -> RF_Module:ESP32-WROOM-32U
- U4: value (none) -> 82400152; footprint (none) -> Package_TO_SOT_SMD:SOT-563
