File: hardware/esp32-spi-hub.kicad_pcb (KiCad board)
At the start: 4 copper layers, 66.9 x 40 mm, 127 parts, among them J1 EXT_HEADER, J2 SM07B-GHS-TB, J3 SM07B-GHS-TB, J4 SM07B-GHS-TB, J5 SM07B-GHS-TB, J6 SM07B-GHS-TB, J7 SM07B-GHS-TB, P1 USB_C_Plug_USB2.0, Q1 AO3401A, Q2 S8050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

Commit message: Add JLCJLCJLCJLC on silkscreen for part number removal
Other:
- board text added: "JLCJLCJLCJLC"
Changed lines of the file:
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@@
     (effects (font (size 0.8 0.8) (thickness 0.1)))
+  )
+  (gr_text "JLCJLCJLCJLC" (at 187.3 123.7 90) (layer "F.SilkS")
+    (effects (font (size 1 1) (thickness 0.15)))
   )
   (gr_text "0" (at 169.8 109.7) (layer "F.SilkS")
